File: hardware/picoavr.sch (EAGLE design)
At the start: 26 parts, among them IC1 MCP1703CB, Q2 12mhz, SW1 SPST_TACT-KMR2, U3 ATMEGA328P, X1 Micro USB

Commit message: add missing labels
Other:
- note added: "1.2"
- note removed: "1.0"
Changed lines of the file:
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@@
 <grid distance="0.1" unitdist="inch" unit="inch" style="lines" multiple="1" display="no" altdistance="0.01" altunitdist="inch" altunit="inch"/>
 <layers>
-<layer number="1" name="Top" color="4" fill="1" visible="yes" active="no"/>
-<layer number="2" name="Route2" color="1" fill="3" visible="yes" active="no"/>
-<layer number="3" name="Route3" color="4" fill="3" visible="yes" active="no"/>
-<layer number="4" name="Route4" color="1" fill="4" visible="yes" active="no"/>
-<layer number="5" name="Route5" color="4" fill="4" visible="yes" active="no"/>
-<layer number="6" name="Route6" color="1" fill="8" visible="yes" active="no"/>
-<layer number="7" name="Route7" color="4" fill="8" visible="yes" active="no"/>
-<layer number="8" name="Route8" color="1" fill="2" visible="yes" active="no"/>
-<layer number="9" name="Route9" color="4" fill="2" visible="yes" active="no"/>
-<layer number="10" name="Route10" color="1" fill="7" visible="yes" active="no"/>
-<layer number="11" name="Route11" color="4" fill="7" visible="yes" active="no"/>
-<layer number="12" name="Route12" color="1" fill="5" visible="yes" active="no"/>
-<layer number="13" name="Route13" color="4" fill="5" visible="yes" active="no"/>
-<layer number="14" name="Route14" color="1" fill="6" visible="yes" active="no"/>
-<layer number="15" name="Route15" color="4" fill="6" visible="yes" active="no"/>
-<layer number="16" name="Bottom" color="1" fill="1" visible="yes" active="no"/>
-<layer number="17" name="Pads" color="2" fill="1" visible="yes" active="no"/>
-<layer number="18" name="Vias" color="2" fill="1" visible="yes" active="no"/>
-<layer number="19" name="Unrouted" color="6" fill="1" visible="yes" active="no"/>
-<layer number="20" name="Dimension" color="15" fill="1" visible="yes" active="no"/>
-<layer number="21" name="tPlace" color="7" fill="1" visible="yes" active="no"/>
-<layer number="22" name="bPlace" color="7" fill="1" visible="yes" active="no"/>
-<layer number="23" name="tOrigins" color="15" fill="1" visible="yes" active="no"/>
-<layer number="24" name="bOrigins" color="15" fill="1" visible="yes" active="no"/>
-<layer number="25" name="tNames" color="7" fill="1" visible="yes" active="no"/>
-<layer number="26" name="bNames" color="7" fill="1" visible="yes" active="no"/>
-<layer number="27" name="tValues" color="7" fill="1" visible="yes" active="no"/>
-<layer number="28" name="bValues" color="7" fill="1" visible="yes" active="no"/>
+<layer number="1" name="Top" color="4" fill="1" visible="no" active="no"/>
+<layer number="2" name="Route2" color="1" fill="3" visible="no" active="no"/>
+<layer number="3" name="Route3" color="4" fill="3" visible="no" active="no"/>
+<layer number="4" name="Route4" color="1" fill="4" visible="no" active="no"/>
+<layer number="5" name="Route5" color="4" fill="4" visible="no" active="no"/>
+<layer number="6" name="Route6" color="1" fill="8" visible="no" active="no"/>
+<layer number="7" name="Route7" color="4" fill="8" visible="no" active="no"/>
+<layer number="8" name="Route8" color="1" fill="2" visible="no" active="no"/>
+<layer number="9" name="Route9" color="4" fill="2" visible="no" active="no"/>
+<layer number="10" name="Route10" color="1" fill="7" visible="no" active="no"/>
+<layer number="11" name="Route11" color="4" fill="7" visible="no" active="no"/>
+<layer number="12" name="Route12" color="1" fill="5" visible="no" active="no"/>
+<layer number="13" name="Route13" color="4" fill="5" visible="no" active="no"/>
+<layer number="14" name="Route14" color="1" fill="6" visible="no" active="no"/>
+<layer number="15" name="Route15" color="4" fill="6" visible="no" active="no"/>
+<layer number="16" name="Bottom" color="1" fill="1" visible="no" active="no"/>
+<layer number="17" name="Pads" color="2" fill="1" visible="no" active="no"/>
+<layer number="18" name="Vias" color="2" fill="1" visible="no" active="no"/>
+<layer number="19" name="Unrouted" color="6" fill="1" visible="no" active="no"/>
+<layer number="20" name="Dimension" color="15" fill="1" visible="no" active="no"/>
+<layer number="21" name="tPlace" color="7" fill="1" visible="no" active="no"/>
+<layer number="22" name="bPlace" color="7" fill="1" visible="no" active="no"/>
+<layer number="23" name="tOrigins" color="15" fill="1" visible="no" active="no"/>
+<layer number="24" name="bOrigins" color="15" fill="1" visible="no" active="no"/>
+<layer number="25" name="tNames" color="7" fill="1" visible="no" active="no"/>
+<layer number="26" name="bNames" color="7" fill="1" visible="no" active="no"/>
+<layer number="27" name="tValues" color="7" fill="1" visible="no" active="no"/>
+<layer number="28" name="bValues" color="7" fill="1" visible="no" active="no"/>
 <layer number="29" name="tStop" color="7" fill="3" visible="no" active="no"/>
 <layer number="30" name="bStop" color="7" fill="6" visible="no" active="no"/>
@@
 <layer number="35" name="tGlue" color="7" fill="4" visible="no" active="no"/>
 <layer number="36" name="bGlue" color="7" fill="5" visible="no" active="no"/>
-<layer number="37" name="tTest" color="7" fill="1" visible="yes" active="no"/>
-<layer number="38" name="bTest" color="7" fill="1" visible="yes" active="no"/>
+<layer number="37" name="tTest" color="7" fill="1" visible="no" active="no"/>
+<layer number="38" name="bTest" color="7" fill="1" visible="no" active="no"/>
 <layer number="39" name="tKeepout" color="4" fill="11" visible="no" active="no"/>
 <layer number="40" name="bKeepout" color="1" fill="11" visible="no" active="no"/>
@@
 <layer number="44" name="Drills" color="7" fill="1" visible="no" active="no"/>
 <layer number="45" name="Holes" color="7" fill="1" visible="no" active="no"/>
-<layer number="46" name="Milling" color="3" fill="1" visible="yes" active="no"/>
-<layer number="47" name="Measures" color="7" fill="1" visible="yes" active="no"/>
-<layer number="48" name="Document" color="7" fill="1" visible="yes" active="no"/>
-<layer number="49" name="Reference" color="7" fill="1" visible="yes" active="no"/>
-<layer number="50" name="dxf" color="7" fill="1" visible="yes" active="no"/>
-<layer number="51" name="tDocu" color="7" fill="1" visible="yes" active="no"/>
-<layer number="52" name="bDocu" color="7" fill="1" visible="yes" active="no"/>
-<layer number="53" name="tGND_GNDA" color="7" fill="9" visible="yes" active="no"/>
-<layer number="54" name="bGND_GNDA" color="1" fill="9" visible="yes" active="no"/>
-<layer number="56" name="wert" color="7" fill="1" visible="yes" active="no"/>
-<layer number="57" name="tCAD" color="7" fill="1" visible="yes" active="no"/>
+<layer number="46" name="Milling" color="3" fill="1" visible="no" active="no"/>
+<layer number="47" name="Measures" color="7" fill="1" visible="no" active="no"/>
+<layer number="48" name="Document" color="7" fill="1" visible="no" active="no"/>
+<layer number="49" name="Reference" color="7" fill="1" visible="no" active="no"/>
+<layer number="50" name="dxf" color="7" fill="1" visible="no" active="no"/>
+<layer number="51" name="tDocu" color="7" fill="1" visible="no" active="no"/>
+<layer number="52" name="bDocu" color="7" fill="1" visible="no" active="no"/>
+<layer number="53" name="tGND_GNDA" color="7" fill="9" visible="no" active="no"/>
+<layer number="54" name="bGND_GNDA" color="1" fill="9" visible="no" active="no"/>
+<layer number="56" name="wert" color="7" fill="1" visible="no" active="no"/>
+<layer number="57" name="tCAD" color="7" fill="1" visible="no" active="no"/>
 <layer number="91" name="Nets" color="2" fill="1" visible="yes" active="yes"/>
 <layer number="92" name="Busses" color="1" fill="1" visible="yes" active="yes"/>
@@
 <description>Rev 1.0</description>
 <plain>
-<text x="99.06" y="12.7" size="1.778" layer="91">1.0</text>
+<text x="99.06" y="12.7" size="1.778" layer="91">1.2</text>
 </plain>
 <instances>
@@
 <pinref part="JSP" gate="G$1" pin="6"/>
 <wire x1="236.22" y1="7.62" x2="241.3" y2="7.62" width="0.1524" layer="91"/>
+<label x="238.76" y="7.62" size="1.778" layer="95"/>
 </segment>
 <segment>
@@
 <pinref part="JSP" gate="G$1" pin="4"/>
 <wire x1="236.22" y1="10.16" x2="241.3" y2="10.16" width="0.1524" layer="91"/>
+<label x="238.76" y="10.16" size="1.778" layer="95"/>
 </segment>
 <segment>
@@
 <pinref part="JSP" gate="G$1" pin="1"/>
 <wire x1="220.98" y1="12.7" x2="218.44" y2="12.7" width="0.1524" layer="91"/>
+<label x="215.9" y="12.7" size="1.778" layer="95"/>
 </segment>
 <segment>
@@
 <pinref part="JSP" gate="G$1" pin="3"/>
 <wire x1="220.98" y1="10.16" x2="218.44" y2="10.16" width="0.1524" layer="91"/>
+<label x="215.9" y="10.16" size="1.778" layer="95"/>
 </segment>
 <segment>
@@
 <pinref part="JSP" gate="G$1" pin="5"/>
 <wire x1="220.98" y1="7.62" x2="218.44" y2="7.62" width="0.1524" layer="91"/>
+<label x="215.9" y="7.62" size="1.778" layer="95"/>
 </segment>
 <segment>
@@
 <pinref part="JP3" gate="G$1" pin="8"/>
 <wire x1="223.52" y1="86.36" x2="231.14" y2="86.36" width="0.1524" layer="91"/>
+<label x="206.756" y="76.2" size="1.778" layer="95"/>
 </segment>
 <segment>
@@
 <pinref part="JP3" gate="G$1" pin="7"/>
 <wire x1="228.6" y1="88.9" x2="231.14" y2="88.9" width="0.1524" layer="91"/>
+<label x="207.01" y="73.66" size="1.778" layer="95"/>
 </segment>
 <segment>
@@
 <pinref part="X1" gate="G$1" pin="VBUS"/>
 <wire x1="14.986" y1="144.018" x2="50.546" y2="144.018" width="0.1524" layer="91"/>
+<label x="40.64" y="144.78" size="1.778" layer="95"/>
 </segment>
 <segment>
@@
 <pinref part="JSP" gate="G$1" pin="2"/>
 <wire x1="236.22" y1="12.7" x2="241.3" y2="12.7" width="0.1524" layer="91"/>
-</segment>
-<segment>
+<label x="238.76" y="12.7" size="1.778" layer="95"/>
+</segment>
+<segment>

Commit message: new hardware revision
Parts:
- removed POWER: (no value), SparkFun-Connectors:M031X03_NO_SILK
- removed R9: 220, SparkFun:RESISTOR0402-RES
- added R4: 10k, resistor:R-US_R0402
- R1, R2: value 4.7k -> 68; device SparkFun:RESISTOR0402-RES -> resistor:R-US_R0402
- R3: value 68 -> 1.5k
- R5: value 68 -> 220; device resistor:R-US_R0402 -> SparkFun:RESISTOR0402-RES
- R6: value 10k -> 4.7k; device resistor:R-US_R0402 -> SparkFun:RESISTOR0402-RES
- R7: value 1.5k -> 4.7k; device resistor:R-US_R0402 -> SparkFun:RESISTOR0402-RES
- renumbered LED2 to LED
Connections:
- net N$11: now also R5.2; no longer R9.2
- net N$2: now also R1.1; no longer R5.1
- net N$4: now also R2.1; no longer R7.1
- net RESET: now also R4.2; no longer R6.2
- net SCK: now also R5.1; no longer R9.1
- net SCL: now also R7.2; no longer R2.2
- net SDA: now also R6.2; no longer R1.2
- net USB_DMINUS: now also R2.2; no longer R3.2
- net USB_DPLUS: now also R1.2; no longer R5.2
- net USB_VBUS: no longer POWER.1
- net VCC: now also R3.2, R4.1, R7.1; no longer POWER.3, R1.1, R2.1, R7.2
- net VPROG: no longer POWER.2
Other:
- moved on the sheet: R1, R2, R3, R5, R6, R7

Commit message: tweaked dimensions
Parts:
- JSP: value (none) -> ICSP
Changed lines of the file:
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@@
 <part name="GND7" library="SparkFun" deviceset="GND" device=""/>
 <part name="R4" library="resistor" deviceset="R-US_" device="R0402" value="10k"/>
-<part name="JSP" library="SparkFun-Connectors" deviceset="M03X2" device="NO_SILK"/>
+<part name="JSP" library="SparkFun-Connectors" deviceset="M03X2" device="NO_SILK" value="ICSP"/>
 <part name="IC1" library="linear" deviceset="MCP1703" device="CB"/>
 <part name="JP2" library="SparkFun-Connectors" deviceset="M14" device="LOCK" value="M14LOCK"/>
